File: linuxpocket.kicad/linuxpocket.kicad_pcb_largebott.kicad_pcb (KiCad board)
At the start: 4 copper layers, 84 x 74.5 mm, 95 parts, among them J1 XDSM-1035-08-KT, J2 Bus_PCI_Express_Mini, J3 HDMI_C_1.4, J4 USB_C_Receptacle_USB2.0_14P, Q1 MMBT3904, SW1 PUSH, SW2 PUSH, SW3 PUSH, U1 BQ24295RGER, U2 BQ27426YZFR, U3 TPS63805YFFR, U4 TPS61169DCKR, U5 MT3608L, U6 FUSB302BUCX, U7 BBQ10KBD, U8 ATmega32U4-M, U9 LIS2MDL

Commit message: PCB almost done and schematic finished.
Parts:
- removed GND, VBAT: TestPoint_Pad_D2.0mm, TestPoint:TestPoint_Pad_D2.0mm
- removed L3, L4: 4.7uH, linuxpocket:IND-SMD_L7.1-W6.6_SL0624
- removed R7: 15k, Resistor_SMD:R_0402_1005Metric
- removed R8: 10k, Resistor_SMD:R_0402_1005Metric
- added D1: LED, Inductor_SMD:L_0603_1608Metric_Pad1.05x0.95mm_HandSolder, F.Cu at (21.6, 122.4)
- added R17: 10k, Resistor_SMD:R_0402_1005Metric, F.Cu at (27.2, 124.1)
- added R5: 10k, Resistor_SMD:R_0402_1005Metric, F.Cu at (20.8, 124.6)
- moved R16 104.1 mm to (27.2, 122.1)
- moved TP4 94.3 mm to (35.8, 169.3)
- moved TP3 90.9 mm to (35.8, 166.3)
- moved TP1 89.9 mm to (35.9, 159.3)
- moved C20 88.5 mm to (162.4, 129.5), turned to 0 degrees
- moved TP2 87.4 mm to (36.1, 163.5)
- moved R20 85.0 mm to (163.0, 142.2), turned to 0 degrees
- moved R19 84.2 mm to (163.2, 136.8), turned to 0 degrees
- moved U5 74.9 mm to (154.2, 139.9)
- moved C18 73.4 mm to (158.1, 114.6)
- moved D3 73.2 mm to (156.9, 132.7), turned to 0 degrees
- moved D2 69.4 mm to (161.7, 115.7), turned to 0 degrees
- moved C21 69.3 mm to (154.8, 136.4), turned to -90 degrees
- moved U4 67.6 mm to (155.3, 115.7), turned to 90 degrees
- moved C19 64.6 mm to (158.1, 116.6)
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- renumbered RS to TP1, SC to TP2, MO to TP3, MI to TP4
Connections:
- J2 pad 17: /GPIO/RI -> /High Speed/RI
- Module1 pad 41: /GPIO/RI -> /GPIO/USB-INT
- Module1 pad 47: /GPIO/MAG_INT -> unconnected-(Module1A-GPIO23-Pad47)
- R16 pad 1: Net-(U2-BIN) -> +1V8
- R16 pad 2: GND -> /High Speed/I^{2}C_SCL
- R25 pad 2: /hs_io/INT -> /GPIO/USB-INT
- U2 pad B1: Net-(U2-BIN) -> unconnected-(U2-BIN-PadB1)
- U6 pad B2: /hs_io/INT -> /GPIO/USB-INT
- U8 pad 1: Net-(Q1-B) -> /GPIO/VOL_DOWN
- U8 pad 10: /Keyboard/MOSI -> unconnected-(U8-PB2-Pad10)
- U8 pad 11: /Keyboard/MISO -> unconnected-(U8-PB3-Pad11)
- U8 pad 18: /GPIO/VOL_DOWN -> Net-(Q1-B)
- U8 pad 19: unconnected-(U8-PD1-Pad19) -> Net-(U7-COL4)
- U8 pad 20: unconnected-(U8-PD2-Pad20) -> Net-(U7-COL5)
- U8 pad 21: unconnected-(U8-PD3-Pad21) -> Net-(U7-ROW3)
- U8 pad 22: unconnected-(U8-PD5-Pad22) -> Net-(U7-ROW4)
- U8 pad 25: Net-(U7-COL4) -> Net-(U7-ROW5)
- U8 pad 26: Net-(U7-ROW3) -> Net-(U7-ROW6)
- U8 pad 27: Net-(U7-COL5) -> Net-(U7-ROW7)
- U8 pad 28: Net-(U7-ROW4) -> Net-(U7-COL1)
- U8 pad 29: Net-(U7-ROW5) -> Net-(U7-COL2)
- U8 pad 30: Net-(U7-ROW6) -> Net-(U7-COL3)
- U8 pad 31: Net-(U7-ROW7) -> Net-(U7-ROW1)
- U8 pad 32: unconnected-(U8-PC7-Pad32) -> Net-(U7-ROW2)
- U8 pad 36: Net-(U7-ROW1) -> unconnected-(U8-PF7-Pad36)
- U8 pad 37: Net-(U7-COL1) -> unconnected-(U8-PF6-Pad37)
- U8 pad 38: Net-(U7-ROW2) -> unconnected-(U8-PF5-Pad38)
- U8 pad 39: Net-(U7-COL2) -> unconnected-(U8-PF4-Pad39)
- U8 pad 40: Net-(U7-COL3) -> unconnected-(U8-PF1-Pad40)
- U8 pad 9: /Keyboard/SCK -> unconnected-(U8-PB1-Pad9)
Routing:
- net +3V3: track 248.1 -> 18.3 mm, vias 12 -> 0
- net /SDA: track 185.2 -> 3.82 mm, vias 6 -> 0
- net /SCL: track 174.3 -> 3.73 mm, vias 5 -> 0
- net /Battery and Power/GAUGE_GPOUT: track 135.0 -> 1.70 mm, vias 2 -> 0
- net /GPIO/PWR_BUT: track 122.8 -> 0.00 mm, vias 2 -> 0
- net /Battery and Power/CHARGE_INT: track 112.3 -> 1.49 mm, vias 2 -> 0
- net /Battery and Power/3V3 EN: track 110.9 -> 1.20 mm, vias 2 -> 0
- net +5V: track 99.4 -> 12.1 mm, vias 7 -> 0
- net /High Speed/HDMI_HP: track 86.4 -> 2.36 mm, vias 2 -> 0
- net /GPIO/SIM_CLK: track 83.7 -> 1.36 mm, vias 2 -> 0
- net /GPIO/SIM_RST: track 82.5 -> 1.30 mm, vias 2 -> 0
- net /Battery and Power/VBload: track 88.9 -> 14.1 mm, vias 7 -> 0
- net /GPIO/SIM_VPP: track 74.0 -> 0.00 mm, vias 2 -> 0
- net /GPIO/SIM_VCC: track 92.6 -> 19.2 mm, vias 2 -> 0
- net /GPIO/SIM_IO: track 77.3 -> 3.90 mm, vias 2 -> 0
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- removed copper zone on F.Cu, net +5V
- removed copper zone on F.Cu, net Net-(D2-A)
- removed copper zone on F.Cu, net Net-(D3-A)
Other:
- outline, holes or cut-outs redrawn
- board text removed: "KEYBOARD"
- board text removed: "MAGNETOMETER"
