File: linuxpocket.kicad/linuxpocket.kicad_pcb (KiCad board)
At the start: 4 copper layers, 84 x 74.5 mm, 95 parts, among them J1 XDSM-1035-08-KT, J2 Bus_PCI_Express_Mini, J3 HDMI_C_1.4, J4 USB_C_Receptacle_USB2.0_14P, Q1 MMBT3904, SW1 PUSH, SW2 PUSH, SW3 PUSH, U1 BQ24295RGER, U2 BQ27426YZFR, U3 TPS63805YFFR, U4 TPS61169DCKR, U5 MT3608L, U6 FUSB302BUCX, U7 BBQ10KBD, U8 ATmega32U4-M, U9 LIS2MDL

Commit message: PCB basically finished.
Parts:
- removed R25: 4.7k, Resistor_SMD:R_0402_1005Metric
- added REF**: MountingHole_2.7mm_M2.5, MountingHole:MountingHole_2.7mm_M2.5, F.Cu at (128.1, 161.5)
- added REF**: Tooling Hole, linuxpocket:Tooling Hole, F.Cu at (130.2, 135.3)
- added REF**: Tooling Hole, linuxpocket:Tooling Hole, F.Cu at (51.8, 155.7)
- added REF**: Tooling Hole, linuxpocket:Tooling Hole, F.Cu at (65.2, 94.0)
- added REF**: KiCad-Logo_5mm_SilkScreen, Symbol:KiCad-Logo_5mm_SilkScreen, B.Cu at (109.6, 106.8)
- added REF**: xamuel, linuxpocket:xamuel, B.Cu at (90.0, 161.6)
- added REF**: ESD-Logo_8.9x8mm_SilkScreen, Symbol:ESD-Logo_8.9x8mm_SilkScreen, B.Cu at (90.0, 120.6)
- added REF**: OSHW-Logo2_14.6x12mm_SilkScreen, Symbol:OSHW-Logo2_14.6x12mm_SilkScreen, B.Cu at (71.3, 106.2)
- renumbered RS to RST
Connections:
- J2 pad 11: /High Speed/PCIE_CLK_N -> unconnected-(J2-REFCLK--Pad11)
- J2 pad 13: /High Speed/PCIE_CLK_P -> unconnected-(J2-REFCLK+-Pad13)
- J2 pad 22: /High Speed/PCIE_nRST -> unconnected-(J2-~{PERST}-Pad22)
- J2 pad 23: /High Speed/PCIE_RX_P -> unconnected-(J2-PERn0-Pad23)
- J2 pad 25: /High Speed/PCIE_RX_N -> unconnected-(J2-PERp0-Pad25)
- J2 pad 31: /High Speed/PCIE_TX_P -> unconnected-(J2-PETn0-Pad31)
- J2 pad 33: /High Speed/PCIE_TX_N -> unconnected-(J2-PETp0-Pad33)
- J2 pad 7: /High Speed/PCIE_CLK_nREQ -> unconnected-(J2-~{CLKREQ}-Pad7)
- J3 pad 20: (no net) -> GND
- J3 pad 21: (no net) -> GND
- J3 pad 22: (no net) -> GND
- J3 pad 23: (no net) -> GND
Routing:
- net +3V3: track 248.1 -> 365.0 mm, vias 12 -> 16
- net GND: track 0.00 -> 76.8 mm, vias 0 -> 54
- net /Battery and Power/VBUS: track 15.7 -> 86.2 mm, vias 0 -> 6
- net /GPIO/RI: track 0.00 -> 49.5 mm, vias 0 -> 4
- net /hs_io/CC1: track 4.14 -> 23.4 mm, vias 0 -> 2
- net /GPIO/MAG_INT: track 0.00 -> 19.2 mm, vias 0 -> 2
- net /High Speed/HDMI_CLK+: track 83.5 -> 80.2 mm
- net /High Speed/HDMI_CLK-: track 85.3 -> 82.1 mm
- net /GPIO/DPI_D14: track 59.9 -> 60.7 mm
- net /Battery and Power/GAUGE_GPOUT: track 135.0 -> 135.6 mm
- net /GPIO/DPI_D11: track 60.5 -> 61.1 mm
- net /High Speed/HDMI_SDA: track 73.1 -> 73.6 mm
- added copper zone on B.Cu, net GND
- added copper zone on F.Cu, net GND
- added copper zone on In1.Cu, net GND
- added copper zone on In2.Cu, net GND
Other:
- board text added: "2.5 clearence beneath CM"
- board text added: "Licensed under CERN-OHL-S-2"
- board text added: "zPocket"
- board text removed: "1.5 clearence beneath CM"
