File: linuxpocket.kicad/linuxpocket.kicad_pcb (KiCad board)
At the start: 4 copper layers, 84 x 74.5 mm, 103 parts, among them J1 XDSM-1035-08-KT, J2 Bus_PCI_Express_Mini, J3 HDMI_C_1.4, J4 USB_C_Receptacle_USB2.0_14P, Q1 MMBT3904, SW1 PUSH, SW2 PUSH, SW3 PUSH, U1 BQ24295RGER, U2 BQ27426YZFR, U3 TPS63805YFFR, U4 TPS61169DCKR, U5 MT3608L, U6 FUSB302BUCX, U7 BBQ10KBD, U8 ATmega32U4-M, U9 LIS2MDL

Commit message: PCB ordered, updated images
Parts:
- added REF**: OSHW-Certification-Mark-Logo_8x4mm_SilkMask, OSHW_Certification_Mark:OSHW-Certification-Mark-Logo_8x4mm_SilkMask, F.Cu at (89.8, 118.9)
- L3, L4: footprint linuxpocket:IND-SMD_L7.1-W6.6_SL0624 -> linuxpocket:IND-SMD_L7.0-W6.6
